Commit message: Imported upstream version '2.5.18' of 'upstream'

File: gazebo_plugins/test/multi_robot_scenario/xacro/p3dx/battery_block.xacro (robot description, xacro)
@@ -1,5 +1,5 @@
 <?xml version="1.0"?>
 <robot xmlns:xacro="http://ros.org/wiki/xacro">
-  <xacro:property name="M_PI" value="3.1415926535897931" />
+  <property name="M_PI" value="3.1415926535897931" />
   <xacro:macro name="battery_block" params="name parent x y z mass">
   <joint name="${parent}_${name}_joint" type="fixed">

File: gazebo_plugins/test/multi_robot_scenario/xacro/p3dx/inertia_tensors.xacro (robot description, xacro)
@@ -4,5 +4,5 @@
   see http://answers.gazebosim.org/question/4372/the-inertia-matrix-explained/ -->
 <robot xmlns:xacro="http://ros.org/wiki/xacro">
-  <xacro:property name="M_PI" value="3.1415926535897931" />
+  <property name="M_PI" value="3.1415926535897931" />
   <!-- see https://secure.wikimedia.org/wikipedia/en/wiki/List_of_moment_of_inertia_tensors -->
   <!-- #################### versions without origin #################### -->
@@ -38,5 +38,5 @@
     <inertial>
       <mass value="${mass}" />
-      <xacro:insert_block name="origin" />
+      <insert_block name="origin" />
       <inertia ixx="${0.4 * mass * radius * radius}" ixy="0.0" ixz="0.0"
         iyy="${0.4 * mass * radius * radius}" iyz="0.0"
@@ -47,5 +47,5 @@
     <inertial>
       <mass value="${mass}" />
-      <xacro:insert_block name="origin" />
+      <insert_block name="origin" />
       <inertia ixx="${0.0833333 * mass * (3 * radius * radius + length * length)}" ixy="0.0" ixz="0.0"
         iyy="${0.0833333 * mass * (3 * radius * radius + length * length)}" iyz="0.0"
@@ -56,5 +56,5 @@
     <inertial>
       <mass value="${mass}" />
-      <xacro:insert_block name="origin" />
+      <insert_block name="origin" />
       <inertia ixx="${0.0833333 * mass * (y*y + z*z)}" ixy="0.0" ixz="0.0"
         iyy="${0.0833333 * mass * (x*x + z*z)}" iyz="0.0"

File: gazebo_plugins/test/multi_robot_scenario/xacro/p3dx/pioneer3dx_chassis.xacro (robot description, xacro)
@@ -1,5 +1,5 @@
 <?xml version="1.0"?>
 <robot xmlns:xacro="http://ros.org/wiki/xacro">
-  <xacro:property name="M_PI" value="3.1415926535897931" />
+  <property name="M_PI" value="3.1415926535897931" />
   <xacro:macro name="pioneer_chassis" params="name parent xyz rpy meshes">
   <!-- Chassis -->

File: gazebo_plugins/test/multi_robot_scenario/xacro/p3dx/pioneer3dx_sonar.xacro (robot description, xacro)
@@ -1,5 +1,5 @@
 <?xml version="1.0"?>
 <robot xmlns:xacro="http://ros.org/wiki/xacro">
-  <xacro:property name="M_PI" value="3.1415926535897931" />
+  <property name="M_PI" value="3.1415926535897931" />
   <xacro:macro name="pioneer_sonar" params="name parent xyz rpy meshes">
   <!-- Front Sonar -->

File: gazebo_plugins/test/multi_robot_scenario/xacro/p3dx/pioneer3dx_swivel.xacro (robot description, xacro)
@@ -1,5 +1,5 @@
 <?xml version="1.0"?>
 <robot xmlns:xacro="http://ros.org/wiki/xacro">
-  <xacro:property name="M_PI" value="3.1415926535897931" />
+  <property name="M_PI" value="3.1415926535897931" />
   <xacro:macro name="pioneer_swivel" params="parent xyz rpy meshes">
   <!-- Swivel -->

File: gazebo_plugins/test/multi_robot_scenario/xacro/p3dx/pioneer3dx_wheel.xacro (robot description, xacro)
@@ -2,5 +2,5 @@
 <robot
   xmlns:xacro="http://ros.org/wiki/xacro">
-  <xacro:property name="M_PI" value="3.1415926535897931" />
+  <property name="M_PI" value="3.1415926535897931" />
   <xacro:macro name="pioneer_wheel" params="side parent xyz rpy radius meshes">
   <!-- Hubcap -->

File: gazebo_plugins/test/tricycle_drive/xacro/tricycle/inertia_tensors.xacro (robot description, xacro)
@@ -4,5 +4,5 @@
   see http://answers.gazebosim.org/question/4372/the-inertia-matrix-explained/ -->
 <robot xmlns:xacro="http://ros.org/wiki/xacro">
-  <xacro:property name="M_PI" value="3.1415926535897931" />
+  <property name="M_PI" value="3.1415926535897931" />
   <!-- see https://secure.wikimedia.org/wikipedia/en/wiki/List_of_moment_of_inertia_tensors -->
   <!-- #################### versions without origin #################### -->
@@ -38,5 +38,5 @@
     <inertial>
       <mass value="${mass}" />
-      <xacro:insert_block name="origin" />
+      <insert_block name="origin" />
       <inertia ixx="${0.4 * mass * radius * radius}" ixy="0.0" ixz="0.0"
         iyy="${0.4 * mass * radius * radius}" iyz="0.0"
@@ -47,5 +47,5 @@
     <inertial>
       <mass value="${mass}" />
-      <xacro:insert_block name="origin" />
+      <insert_block name="origin" />
       <inertia ixx="${0.0833333 * mass * (3 * radius * radius + length * length)}" ixy="0.0" ixz="0.0"
         iyy="${0.0833333 * mass * (3 * radius * radius + length * length)}" iyz="0.0"

File: gazebo_plugins/test/tricycle_drive/xacro/tricycle/tricycle_body.xacro (robot description, xacro)
@@ -1,7 +1,7 @@
 <?xml version="1.0"?>
 <robot xmlns:xacro="http://www.ros.org/wiki/xacro">
-  <xacro:property name="M_PI" value="3.1415926535897931" />
-  <xacro:property name="radius_actuated_wheel" value="0.135" />
-  <xacro:property name="radius_encoder_wheel" value="0.135" />
+  <property name="M_PI" value="3.1415926535897931" />
+  <property name="radius_actuated_wheel" value="0.135" />
+  <property name="radius_encoder_wheel" value="0.135" />
   <xacro:include filename="inertia_tensors.xacro"/>
   <xacro:include filename="tricycle_chassis.xacro"/>

File: gazebo_plugins/test/tricycle_drive/xacro/tricycle/tricycle_chassis.xacro (robot description, xacro)
@@ -1,8 +1,8 @@
 <?xml version="1.0"?>
 <robot xmlns:xacro="http://ros.org/wiki/xacro">
-  <xacro:property name="M_PI" value="3.1415926535897931" />
-  <xacro:property name="DX" value="2.500" />
-  <xacro:property name="DY" value="0.60" />
-  <xacro:property name="DZ" value="0.1" />
+  <property name="M_PI" value="3.1415926535897931" />
+  <property name="DX" value="2.500" />
+  <property name="DY" value="0.60" />
+  <property name="DZ" value="0.1" />
   <xacro:macro name="tricycle_chassis" params="name parent xyz rpy meshes">
   <!-- Chassis -->

File: gazebo_plugins/test/tricycle_drive/xacro/tricycle/wheel.xacro (robot description, xacro)
@@ -2,5 +2,5 @@
 <robot
   xmlns:xacro="http://ros.org/wiki/xacro">
-  <xacro:property name="M_PI" value="3.1415926535897931" />
+  <property name="M_PI" value="3.1415926535897931" />
   <xacro:macro name="wheel" params="name parent xyz rpy radius length meshes">
   <!-- Wheel -->

File: gazebo_plugins/test/tricycle_drive/xacro/tricycle/wheel_actuated.xacro (robot description, xacro)
@@ -1,5 +1,5 @@
 <?xml version="1.0"?>
 <robot xmlns:xacro="http://ros.org/wiki/xacro">
-  <xacro:property name="M_PI" value="3.1415926535897931" />
+  <property name="M_PI" value="3.1415926535897931" />
   <xacro:macro name="wheel_actuated" params="name parent xyz rpy radius length meshes">
   <!-- steering joint -->

File: gazebo_plugins/test2/large_models/large_model.urdf.xacro (robot description, xacro)
@@ -20,6 +20,6 @@
   <xacro:macro name="one_link" params="link_name parent *axis *origin material">
     <joint name="${link_name}_joint" type="continuous" >
-      <xacro:insert_block name="origin"/>
-      <xacro:insert_block name="axis"/>
+      <insert_block name="origin"/>
+      <insert_block name="axis"/>
       <parent link="${parent}" />
       <child link="${link_name}" />

File: gazebo_plugins/test2/large_models/smaller_large_model.urdf.xacro (robot description, xacro)
@@ -20,6 +20,6 @@
   <xacro:macro name="one_link" params="link_name parent *axis *origin material">
     <joint name="${link_name}_joint" type="continuous" >
-      <xacro:insert_block name="origin"/>
-      <xacro:insert_block name="axis"/>
+      <insert_block name="origin"/>
+      <insert_block name="axis"/>
       <parent link="${parent}" />
       <child link="${link_name}" />
